File: thermostat.kicad_pcb (KiCad board)
At the start: 2 copper layers, 63 x 98 mm, 76 parts, among them J1 Rc/C, J3 I2C, J4 Outputs G/OB, J5 Outputs W1/W2/E/Rh, J6 Xiao1, J7 Xiao2, J8 Outdoor DS18B20, J9 Dial 5V, Q1 BT138-600E, Q2 BT138-600E, Q3 BT138-600E, Q4 BT138-600E, Q5 BT138-600E, Q6 BT138-600E, Q7 BT138-600E, Q8 TIP122, U1 K7805-500R3, U10 MOC3063, U3 DS18B20, U4 MOC3063, U5 MOC3063, U6 MOC3063, U7 MOC3063, U8 MOC3063, U9 MOC3063

Commit message: Update for JLC order: C2 5 mm, U3 power fix, new BOMs, 1.1 mm header holes
- C2 footprint is now 5.00 mm pitch; fab files and CPL regenerated
  (fab zip 2026-10-25 matches the boards ordered from JLC)
- Schematic: move U3's +3V3 and GND symbols back onto its wires
- BOM-LCSC.csv reformatted (Comment/Designator/Footprint/.../Notes);
  new BOM-JLC.csv and BOM-NextPCB.xls (one row per part)
- PCB: header drills (J3, J6, J7, J9, JP1) 1.0 -> 1.1 mm for the next
  revision; fab files were NOT regenerated for this change

Co-Authored-By: Claude Sonnet 5.5 <noreply@anthropic.com>
Claude-Session: https://claude.ai/code/session_01E7T4v2apyDnHDNPi6eHwQU
Parts:
- C2: footprint Capacitor_THT:C_Disc_D5.0mm_W2.5mm_P2.50mm -> Capacitor_THT:C_Disc_D5.0mm_W2.5mm_P5.00mm
- D10: value BZX79-C30 -> BZX55C30
- moved C2 1.35 mm to (80.5, 139.0)
